File: python/templates/template_with_symbols.kicad_sch (KiCad schematic)
At the start: 3 parts

Commit message: fix: Update schematic format to KiCAD 9 and fix invalid UUIDs (#37)
- Update schematic version from 20230121 (KiCAD 7) to 20240101 (KiCAD 9)
- Replace invalid all-zeros UUIDs in template files with valid UUIDs
- Add post-copy UUID regeneration to ensure each project gets unique UUID
- Add UTF-8 encoding and Unix line endings for cross-platform compatibility

Fixes the root cause where templates were copied with invalid UUIDs and
outdated version format, causing KiCAD 9.0.x to reject the schematic files.

Co-Authored-By: Claude Opus 4.6 <noreply@anthropic.com>
Connections:
- net at _TEMPLATE_R.1: no longer _TEMPLATE_C.1
- net at _TEMPLATE_R.2: no longer _TEMPLATE_C.2
Other:
- moved on the sheet: _TEMPLATE_C, _TEMPLATE_D, _TEMPLATE_R
Changed lines of the file:
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@@
-(kicad_sch (version 20250114) (generator "KiCAD-MCP-Server")
+(kicad_sch (version 20240101) (generator "KiCAD-MCP-Server")
   (paper "A4")
-  (symbol (lib_id "Device:R") (at -10000 -10000 0) (unit 1)
+  (symbol (lib_id "Device:R") (at -100 -100 0) (unit 1)
     (in_bom no) (on_board no) (dnp yes)
     (property "Reference" "_TEMPLATE_R" (at -100 -102.54 0)
@@
       (effects (font (size 1.27 1.27)) hide)
     )
-    (property "Datasheet" "~" (at -10000 -10000 0)
+    (property "Datasheet" "~" (at -100 -100 0)
       (effects (font (size 1.27 1.27)) hide)
     )
@@
     (pin "2")
   )
-  (symbol (lib_id "Device:C") (at -10000 -10000 0) (unit 1)
+  (symbol (lib_id "Device:C") (at -100 -110 0) (unit 1)
     (in_bom no) (on_board no) (dnp yes)
     (property "Reference" "_TEMPLATE_C" (at -100 -107.46 0)
@@
       (effects (font (size 1.27 1.27)))
     )
-    (property "Footprint" "" (at -10000 -10000 0)
+    (property "Footprint" "" (at -100 -110 0)
       (effects (font (size 1.27 1.27)) hide)
     )
-    (property "Datasheet" "~" (at -10000 -10000 0)
+    (property "Datasheet" "~" (at -100 -110 0)
       (effects (font (size 1.27 1.27)) hide)
     )
@@
     (pin "2")
   )
-  (symbol (lib_id "Device:LED") (at -10000 -10000 0) (unit 1)
+  (symbol (lib_id "Device:LED") (at -100 -120 0) (unit 1)
     (in_bom no) (on_board no) (dnp yes)
     (property "Reference" "_TEMPLATE_D" (at -100 -117.46 0)
@@
       (effects (font (size 1.27 1.27)))
     )
-    (property "Footprint" "" (at -10000 -10000 0)
+    (property "Footprint" "" (at -100 -120 0)
       (effects (font (size 1.27 1.27)) hide)
     )
-    (property "Datasheet" "~" (at -10000 -10000 0)
+    (property "Datasheet" "~" (at -100 -120 0)
       (effects (font (size 1.27 1.27)) hide)
     )
