File: python/templates/template_with_symbols_expanded.kicad_sch (KiCad schematic)
At the start: 0 parts

Commit message: fix: Update schematic format to KiCAD 9 and fix invalid UUIDs (#37)
- Update schematic version from 20230121 (KiCAD 7) to 20240101 (KiCAD 9)
- Replace invalid all-zeros UUIDs in template files with valid UUIDs
- Add post-copy UUID regeneration to ensure each project gets unique UUID
- Add UTF-8 encoding and Unix line endings for cross-platform compatibility

Fixes the root cause where templates were copied with invalid UUIDs and
outdated version format, causing KiCAD 9.0.x to reject the schematic files.

Co-Authored-By: Claude Opus 4.6 <noreply@anthropic.com>
Parts:
- added _TEMPLATE_C: C, symbol Device:C
- added _TEMPLATE_D: D, symbol Device:D
- added _TEMPLATE_J2: Conn_2, symbol Connector_Generic:Conn_01x02
- added _TEMPLATE_J4: Conn_4, symbol Connector_Generic:Conn_01x04
- added _TEMPLATE_L: L, symbol Device:L
- added _TEMPLATE_LED: LED, symbol Device:LED
- added _TEMPLATE_Q_NMOS: Q_NMOS, symbol Device:Q_NMOS_GSD
- added _TEMPLATE_Q_NPN: Q_NPN, symbol Device:Q_NPN_BCE
- added _TEMPLATE_R: R, symbol Device:R
- added _TEMPLATE_SW: Switch, symbol Switch:SW_Push
- added _TEMPLATE_U_OPAMP: OpAmp, symbol Amplifier_Operational:LM358
- added _TEMPLATE_U_REG: Regulator, symbol Regulator_Linear:AMS1117-3.3
- added _TEMPLATE_Y: Crystal, symbol Device:Crystal
Changed lines of the file:
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@@
-(kicad_sch (version 20250114) (generator "KiCAD-MCP-Server")
+(kicad_sch (version 20240101) (generator "KiCAD-MCP-Server")
   (paper "A4")
+  ;; TEMPLATE INSTANCES (placed offscreen at -100, -110, etc.)
+  (symbol (lib_id "Device:R") (at -100 -100 0) (unit 1)
+    (in_bom no) (on_board no) (dnp yes)
+    (property "Reference" "_TEMPLATE_R" (at -100 -102.54 0)
+      (effects (font (size 1.27 1.27)))
+    )
+    (property "Value" "R" (at -100 -100 90)
+      (effects (font (size 1.27 1.27)))
+    )
+    (property "Footprint" "" (at -100 -100 90)
+      (effects (font (size 1.27 1.27)) hide)
+    )
+    (property "Datasheet" "~" (at -100 -100 0)
+      (effects (font (size 1.27 1.27)) hide)
+    )
+    (pin "1")
+    (pin "2")
+  )
+  (symbol (lib_id "Device:C") (at -100 -110 0) (unit 1)
+    (in_bom no) (on_board no) (dnp yes)
+    (property "Reference" "_TEMPLATE_C" (at -100 -107.46 0)
+      (effects (font (size 1.27 1.27)))
+    )
+    (property "Value" "C" (at -100 -112.54 0)
+      (effects (font (size 1.27 1.27)))
+    )
+    (property "Footprint" "" (at -100 -110 0)
+      (effects (font (size 1.27 1.27)) hide)
+    )
+    (property "Datasheet" "~" (at -100 -110 0)
+      (effects (font (size 1.27 1.27)) hide)
+    )
+    (pin "1")
+    (pin "2")
+  )
+  (symbol (lib_id "Device:L") (at -100 -120 0) (unit 1)
+    (in_bom no) (on_board no) (dnp yes)
+    (property "Reference" "_TEMPLATE_L" (at -100 -117.46 0)
+      (effects (font (size 1.27 1.27)))
+    )
+    (property "Value" "L" (at -100 -122.54 0)
+      (effects (font (size 1.27 1.27)))
+    )
+    (property "Footprint" "" (at -100 -120 0)
+      (effects (font (size 1.27 1.27)) hide)
+    )
+    (property "Datasheet" "~" (at -100 -120 0)
+      (effects (font (size 1.27 1.27)) hide)
+    )
+    (pin "1")
+    (pin "2")
+  )
+  (symbol (lib_id "Device:Crystal") (at -100 -130 0) (unit 1)
+    (in_bom no) (on_board no) (dnp yes)
+    (property "Reference" "_TEMPLATE_Y" (at -100 -127.46 0)
+      (effects (font (size 1.27 1.27)))
+    )
+    (property "Value" "Crystal" (at -100 -132.54 0)
+      (effects (font (size 1.27 1.27)))
+    )
+    (property "Footprint" "" (at -100 -130 0)
+      (effects (font (size 1.27 1.27)) hide)
+    )
+    (property "Datasheet" "~" (at -100 -130 0)
+      (effects (font (size 1.27 1.27)) hide)
+    )
+    (pin "1")
+    (pin "2")
+  )
+  (symbol (lib_id "Device:D") (at -100 -140 0) (unit 1)
+    (in_bom no) (on_board no) (dnp yes)
+    (property "Reference" "_TEMPLATE_D" (at -100 -137.46 0)
+      (effects (font (size 1.27 1.27)))
+    )
+    (property "Value" "D" (at -100 -142.54 0)
+      (effects (font (size 1.27 1.27)))
+    )
+    (property "Footprint" "" (at -100 -140 0)
+      (effects (font (size 1.27 1.27)) hide)
+    )
+    (property "Datasheet" "~" (at -100 -140 0)
+      (effects (font (size 1.27 1.27)) hide)
+    )
+    (pin "1")
+    (pin "2")
+  )
+  (symbol (lib_id "Device:LED") (at -100 -150 0) (unit 1)
+    (in_bom no) (on_board no) (dnp yes)
+    (property "Reference" "_TEMPLATE_LED" (at -100 -147.46 0)
+      (effects (font (size 1.27 1.27)))
+    )
+    (property "Value" "LED" (at -100 -152.54 0)
+      (effects (font (size 1.27 1.27)))
+    )
+    (property "Footprint" "" (at -100 -150 0)
+      (effects (font (size 1.27 1.27)) hide)
+    )
+    (property "Datasheet" "~" (at -100 -150 0)
+      (effects (font (size 1.27 1.27)) hide)
+    )
+    (pin "1")
+    (pin "2")
+  )
+  (symbol (lib_id "Device:Q_NPN_BCE") (at -100 -160 0) (unit 1)
+    (in_bom no) (on_board no) (dnp yes)
+    (property "Reference" "_TEMPLATE_Q_NPN" (at -100 -157.46 0)
+      (effects (font (size 1.27 1.27)))
+    )
+    (property "Value" "Q_NPN" (at -100 -162.54 0)
+      (effects (font (size 1.27 1.27)))
+    )
+    (property "Footprint" "" (at -100 -160 0)
+      (effects (font (size 1.27 1.27)) hide)
+    )
+    (property "Datasheet" "~" (at -100 -160 0)
+      (effects (font (size 1.27 1.27)) hide)
+    )
+    (pin "1")
+    (pin "2")
+    (pin "3")
+  )
+  (symbol (lib_id "Device:Q_NMOS_GSD") (at -100 -170 0) (unit 1)
+    (in_bom no) (on_board no) (dnp yes)
+    (property "Reference" "_TEMPLATE_Q_NMOS" (at -100 -167.46 0)
+      (effects (font (size 1.27 1.27)))
+    )
+    (property "Value" "Q_NMOS" (at -100 -172.54 0)
+      (effects (font (size 1.27 1.27)))
+    )
+    (property "Footprint" "" (at -100 -170 0)
+      (effects (font (size 1.27 1.27)) hide)
+    )
+    (property "Datasheet" "~" (at -100 -170 0)
+      (effects (font (size 1.27 1.27)) hide)
+    )
+    (pin "1")
+    (pin "2")
+    (pin "3")
+  )
+  (symbol (lib_id "Amplifier_Operational:LM358") (at -100 -180 0) (unit 1)
+    (in_bom no) (on_board no) (dnp yes)
+    (property "Reference" "_TEMPLATE_U_OPAMP" (at -100 -177.46 0)
+      (effects (font (size 1.27 1.27)))
+    )
+    (property "Value" "OpAmp" (at -100 -182.54 0)
+      (effects (font (size 1.27 1.27)))
+    )
+    (property "Footprint" "" (at -100 -180 0)
+      (effects (font (size 1.27 1.27)) hide)
+    )
+    (property "Datasheet" "" (at -100 -180 0)
+      (effects (font (size 1.27 1.27)) hide)
+    )
+    (pin "1")
+    (pin "2")
+    (pin "3")
+    (pin "4")
+    (pin "8")
+  )
+  (symbol (lib_id "Connector_Generic:Conn_01x02") (at -100 -190 0) (unit 1)
+    (in_bom no) (on_board no) (dnp yes)
+    (property "Reference" "_TEMPLATE_J2" (at -100 -187.46 0)
+      (effects (font (size 1.27 1.27)))
+    )
+    (property "Value" "Conn_2" (at -100 -192.54 0)
+      (effects (font (size 1.27 1.27)))
+    )
+    (property "Footprint" "" (at -100 -190 0)
+      (effects (font (size 1.27 1.27)) hide)
+    )
+    (property "Datasheet" "~" (at -100 -190 0)
+      (effects (font (size 1.27 1.27)) hide)
+    )
+    (pin "1")
+    (pin "2")
+  )
+  (symbol (lib_id "Connector_Generic:Conn_01x04") (at -100 -200 0) (unit 1)
+    (in_bom no) (on_board no) (dnp yes)
+    (property "Reference" "_TEMPLATE_J4" (at -100 -197.46 0)
+      (effects (font (size 1.27 1.27)))
+    )
+    (property "Value" "Conn_4" (at -100 -202.54 0)
+      (effects (font (size 1.27 1.27)))
+    )
+    (property "Footprint" "" (at -100 -200 0)
+      (effects (font (size 1.27 1.27)) hide)
+    )
+    (property "Datasheet" "~" (at -100 -200 0)
+      (effects (font (size 1.27 1.27)) hide)
+    )
+    (pin "1")
+    (pin "2")
+    (pin "3")
+    (pin "4")
+  )
+  (symbol (lib_id "Regulator_Linear:AMS1117-3.3") (at -100 -210 0) (unit 1)
+    (in_bom no) (on_board no) (dnp yes)
+    (property "Reference" "_TEMPLATE_U_REG" (at -100 -207.46 0)
+      (effects (font (size 1.27 1.27)))
+    )
+    (property "Value" "Regulator" (at -100 -212.54 0)
+      (effects (font (size 1.27 1.27)))
+    )
+    (property "Footprint" "" (at -100 -210 0)
+      (effects (font (size 1.27 1.27)) hide)
+    )
+    (property "Datasheet" "" (at -100 -210 0)
+      (effects (font (size 1.27 1.27)) hide)
+    )
+    (pin "1")
+    (pin "2")
+    (pin "3")
+  )
+  (symbol (lib_id "Switch:SW_Push") (at -100 -220 0) (unit 1)
+    (in_bom no) (on_board no) (dnp yes)
+    (property "Reference" "_TEMPLATE_SW" (at -100 -217.46 0)
+      (effects (font (size 1.27 1.27)))
+    )
+    (property "Value" "Switch" (at -100 -222.54 0)
+      (effects (font (size 1.27 1.27)))
+    )
+    (property "Footprint" "" (at -100 -220 0)
+      (effects (font (size 1.27 1.27)) hide)
+    )
+    (property "Datasheet" "~" (at -100 -220 0)
+      (effects (font (size 1.27 1.27)) hide)
+    )
+    (pin "1")
+    (pin "2")
+  )
   (sheet_instances
     (path "/" (page "1"))
